File: esp32_vtx.kicad_sch (KiCad schematic)
At the start: 33 parts, among them J1 Conn_01x24_MountingPin, J2 Conn_01x05, U1 AMS1117-3.3, U2 IS25WP032, U3 ESP32-PICO-D4, U4 MKDV4GCL-AB, U5 XC6206-2.8V, U6 XC6206-1.2V

Commit message: add cap near pclk, change package of res and cap to 0603
Signed-off-by: huangzzk <huangcmzzk@gmail.com>
Parts:
- added C2: 0.1uF, Capacitor_SMD:C_0603_1608Metric, symbol Device:C
- C10, C11, C15, C5, C6, C9: footprint Capacitor_SMD:C_0402_1005Metric -> Capacitor_SMD:C_0603_1608Metric
- R1, R11, R12, R14, R15, R16, R17, R18, R9: footprint Resistor_SMD:R_0402_1005Metric -> Resistor_SMD:R_0603_1608Metric
Connections:
- net GND: now also C2.2
- net PCLK: now also C2.1

Commit message: changes pclk cap value to 22pf instead of 0.1uF
Signed-off-by: huangzzk <huangcmzzk@gmail.com>
Parts:
- C2: value 0.1uF -> 22pf
Changed lines of the file:
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@@
     (in_bom yes) (on_board yes)
     (property "Reference" "C2" (id 0) (at 45.72 67.945 0))
-    (property "Value" "0.1uF" (id 1) (at 43.18 67.945 0))
+    (property "Value" "22pf" (id 1) (at 43.18 67.945 0))
     (property "Footprint" "Capacitor_SMD:C_0603_1608Metric" (id 2) (at 48.895 63.1698 0)
       (effects (font (size 1.27 1.27)) hide)
@@
     )
     (path "/2fc429b0-8f95-4a55-a702-5f5bc11d40b4"
-      (reference "C2") (unit 1) (value "0.1uF") (footprint "Capacitor_SMD:C_0603_1608Metric")
+      (reference "C2") (unit 1) (value "22pf") (footprint "Capacitor_SMD:C_0603_1608Metric")
     )
     (path "/a350a85d-0544-4287-b9e5-c3217e648cae"

Commit message: v1.1 tested.
Signed-off-by: huangzzk <huangcmzzk@gmail.com>
Parts:
- removed C6: 0.1uF, Capacitor_SMD:C_0603_1608Metric, symbol Device:C
- removed J2: Conn_01x05, Connector_PinHeader_2.54mm:PinHeader_1x05_P2.54mm_Vertical, symbol Connector_Generic:Conn_01x05
- added C3: 100uF, symbol Device:C_Polarized
- added J2: Conn_01x04, Connector_PinHeader_2.54mm:PinHeader_1x04_P2.54mm_Vertical, symbol Connector_Generic:Conn_01x04
- added R2, R3: 0R, Resistor_SMD:R_0603_1608Metric, symbol Device:R
- added SW1, SW2: SW_SPST, Button_Switch_SMD:SW_SPST_B3U-1000P, symbol Switch:SW_SPST
- C2: value 22pf -> 15pF
Connections:
- net +3V3: now also C3.1
- net +5V: now also J2.1 (Pin_1)
- net GND: now also C3.2, J2.4 (Pin_4), R2.2, R3.2, SW1.2 (B), SW2.2 (B); no longer C12.2, C13.2, C14.2, C16.2, C2.2, J1.10 (Pin_10), J1.23 (Pin_23), U5.1 (GND), U6.1 (GND)
- net GPIO0: now also SW2.1 (A)
- net RX: now also J2.3 (Pin_3)
- net TX: now also J2.2 (Pin_2)
- net SD_DATA0 renamed GPIO2
- net GPIO2: now also SW1.1 (A)
- new net GNDA: C13.2, C16.2, J1.23 (Pin_23), R3.1, U5.1 (GND)
- new net GNDD: C12.2, C14.2, C2.2, J1.10 (Pin_10), R2.1, U6.1 (GND)

Commit message: update
Signed-off-by: huangzzk <huangcmzzk@gmail.com>
Parts:
- removed R2, R3: 0R, Resistor_SMD:R_0603_1608Metric, symbol Device:R
- removed RF1: KH-IPEX4-2020, ic_footprint:IPEX4-SMD_4P-L1.8-W1.7-LS2.0-L_KH-IPEX4-2020, symbol ic:KH-IPEX4-2020
- added C17, C18, C19, C4, C6: 10u, Capacitor_SMD:C_0603_1608Metric, symbol Device:C
- added H1, H2, H3, H4: MountingHole, MountingHole:MountingHole_2.2mm_M2, symbol Mechanical:MountingHole
- added RF1: BWIPX-1-001E, kicad_lceda:IPEX-SMD_BWIPX-1-001E, symbol ic:BWIPX-1-001E
- C3: footprint (none) -> Capacitor_Tantalum_SMD:CP_EIA-3216-18_Kemet-A
Connections:
- net GNDA is gone; now on net GND: C13.2, C16.2, J1.23 (Pin_23), U5.1 (GND)
- net GNDD is gone; now on net GND: C12.2, C14.2, C2.2, J1.10 (Pin_10), U6.1 (GND)
- net +3V3: now also C17.1, C18.1, C19.1, C4.1, C6.1
- net GND: now also C17.2, C18.2, C19.2, C4.2, C6.2, RF1.2 (GND), RF1.3 (GND)
- net RFOUT: now also RF1.1 (SIG)
